Commit message: Sawyer xacro, launch and yaml updates
- Adds sawyer_moveit.launch as the default entrypoint for launching
- Adds kinect_sensor and xtion_sensor yaml configs, launch args
- Adds rethink_electric_gripper srdf xacro files for Sawyer
- Adds sawyer srdf xacro files for self collision

File: sawyer_moveit_config/srdf/sawyer_base.srdf.xacro (robot description, xacro)
@@ -1,22 +1,29 @@
 <?xml version="1.0" ?>
 <!--This does not replace URDF, and is not an extension of URDF.
-    This is a format for representing semantic information about the robot structure.
-    A URDF file must exist for this robot as well, where the joints and the links that are referenced are defined
+    This is a format for representing semantic information about the robot
+    structure. A URDF file must exist for this robot as well, where the joints
+    and the links that are referenced are defined
 -->
-<robot name="sawyer">
-    <!--GROUPS: Representation of a set of joints and links. This can be useful for specifying DOF to plan for, defining arms, end effectors, etc-->
-    <!--LINKS: When a link is specified, the parent joint of that link (if it exists) is automatically included-->
-    <!--JOINTS: When a joint is specified, the child link of that joint (which will always exist) is automatically included-->
-    <!--CHAINS: When a chain is specified, all the links along the chain (including endpoints) are included in the group. Additionally, all the joints that are parents to included links are also included. This means that joints along the chain and the parent joint of the base link are included in the group-->
-    <!--SUBGROUPS: Groups can also be formed by referencing to already defined group names-->
+<robot xmlns:xacro="http://www.ros.org/wiki/xacro" name="sawyer">
+  <xacro:macro name="sawyer_base" params="tip_name">
+    <xacro:arg name="tip_name" default="right_hand"/>
+    <!--GROUPS: Representation of a set of joints and links. This can be useful
+    for specifying DOF to plan for, defining arms, end effectors, etc-->
+    <!--LINKS: When a link is specified, the parent joint of that link (if it
+    exists) is automatically included-->
+    <!--JOINTS: When a joint is specified, the child link of that joint (which
+    will always exist) is automatically included-->
+    <!--CHAINS: When a chain is specified, all the links along the chain
+    (including endpoints) are included in the group. Additionally, all the
+    joints that are parents to included links are also included. This means
+    that joints along the chain and the parent joint of the base link are
+    included in the group-->
+    <!--SUBGROUPS: Groups can also be formed by referencing to already defined
+    group names-->
     <group name="right_arm">
-        <chain base_link="base" tip_link="right_hand" />
+        <chain base_link="base" tip_link="$(arg tip_name)" />
     </group>
-    <group name="right_hand">
-        <link name="right_hand" />
-        <link name="right_gripper_base" />
-        <link name="right_gripper" />
-    </group>
-    <!--GROUP STATES: Purpose: Define a named state for a particular group, in terms of joint values. This is useful to define states like 'folded arms'-->
+    <!--GROUP STATES: Purpose: Define a named state for a particular group, in
+    terms of joint values. This is useful to define states like 'folded arms'-->
     <group_state name="zero_pose" group="right_arm">
         <joint name="right_j0" value="0" />
@@ -28,9 +35,11 @@
         <joint name="right_j6" value="0" />
     </group_state>
-    <!--END EFFECTOR: Purpose: Represent information about an end effector.-->
-    <end_effector name="right_hand_eef" parent_link="right_gripper" group="right_hand" parent_group="right_arm" />
-    <!--VIRTUAL JOINT: Purpose: this element defines a virtual joint between a robot link and an external frame of reference (considered fixed with respect to the robot)-->
+    <!--VIRTUAL JOINT: Purpose: this element defines a virtual joint between a
+    robot link and an external frame of reference (considered fixed with
+    respect to the robot)-->
     <virtual_joint name="world" type="fixed" parent_frame="world" child_link="base" />
-    <!--DISABLE COLLISIONS: By default it is assumed that any link of the robot could potentially come into collision with any other link in the robot. This tag disables collision checking between a specified pair of links. -->
+    <!--DISABLE COLLISIONS: By default it is assumed that any link of the robot
+    could potentially come into collision with any other link in the robot.
+    This tag disables collision checking between a specified pair of links. -->
     <disable_collisions link1="head" link2="pedestal" reason="Never" />
     <disable_collisions link1="head" link2="right_arm_base_link" reason="Never" />
@@ -49,18 +58,4 @@
     <disable_collisions link1="right_arm_base_link" link2="screen" reason="Never" />
     <disable_collisions link1="right_arm_base_link" link2="torso" reason="Adjacent" />
-    <disable_collisions link1="right_gripper" link2="right_gripper_base" reason="Adjacent" />
-    <disable_collisions link1="right_gripper" link2="right_hand" reason="Default" />
-    <disable_collisions link1="right_gripper" link2="right_l3" reason="Never" />
-    <disable_collisions link1="right_gripper" link2="right_l4" reason="Never" />
-    <disable_collisions link1="right_gripper" link2="right_l5" reason="Never" />
-    <disable_collisions link1="right_gripper" link2="right_l6" reason="Default" />
-    <disable_collisions link1="right_gripper" link2="screen" reason="Never" />
-    <disable_collisions link1="right_gripper" link2="torso" reason="Never" />
-    <disable_collisions link1="right_gripper_base" link2="right_hand" reason="Adjacent" />
-    <disable_collisions link1="right_gripper_base" link2="right_l3" reason="Never" />
-    <disable_collisions link1="right_gripper_base" link2="right_l4" reason="Never" />
-    <disable_collisions link1="right_gripper_base" link2="right_l5" reason="Never" />
-    <disable_collisions link1="right_gripper_base" link2="right_l6" reason="Default" />
-    <disable_collisions link1="right_gripper_base" link2="screen" reason="Never" />
     <disable_collisions link1="right_hand" link2="right_l3" reason="Never" />
     <disable_collisions link1="right_hand" link2="right_l4" reason="Never" />
@@ -91,3 +86,4 @@
     <disable_collisions link1="right_l5" link2="right_l6" reason="Adjacent" />
     <disable_collisions link1="screen" link2="torso" reason="Never" />
+  </xacro:macro>
 </robot>
