Commit message: Updates for dynamic gripper joints in 5.2
- Updates the xacro for Sawyer SRDF to use dynamic joints
- Update the naming schemes for the electric gripper
- Updates the kinematic chain tips

File: sawyer_moveit_config/srdf/rethink_electric_gripper.srdf.xacro (robot description, xacro)
@@ -6,51 +6,48 @@
 <robot xmlns:xacro="http://www.ros.org/wiki/xacro" name="rethink_electric_gripper">
     <xacro:macro name="rethink_electric_gripper" params="side">
-    <xacro:property name="gripper_side" value="${side[0]}" scope="local"/>
     <disable_collisions link1="${side}_l6" link2="${side}_gripper_base" reason="Adjacent" />
-    <disable_collisions link1="${side}_gripper_base" link2="${side}_gripper" reason="Adjacent" />
-    <disable_collisions link1="${side}_gripper" link2="${side}_hand" reason="Adjacent" />
+    <disable_collisions link1="${side}_gripper_base" link2="${side}_gripper_tip" reason="Adjacent" />
+    <disable_collisions link1="${side}_gripper_tip" link2="${side}_hand" reason="Adjacent" />
     <disable_collisions link1="${side}_hand" link2="${side}_gripper_base" reason="Adjacent" />
-    <xacro:if value="false"> <!-- Add these back in once articulated gripper is available -->
     <disable_collisions link1="${side}_hand" link2="${side}_connector_plate_base" reason="Adjacent" />
     <disable_collisions link1="${side}_hand" link2="${side}_electric_gripper_base" reason="Adjacent" />
-    <disable_collisions link1="${side}_gripper_base" link2="${gripper_side}_gripper_l_finger" reason="Adjacent" />
-    <disable_collisions link1="${side}_gripper_base" link2="${gripper_side}_gripper_l_finger_tip" reason="Never" />
-    <disable_collisions link1="${side}_gripper_base" link2="${gripper_side}_gripper_r_finger" reason="Adjacent" />
-    <disable_collisions link1="${side}_gripper_base" link2="${gripper_side}_gripper_r_finger_tip" reason="Never" />
+    <disable_collisions link1="${side}_gripper_base" link2="${side}_gripper_l_finger" reason="Adjacent" />
+    <disable_collisions link1="${side}_gripper_base" link2="${side}_gripper_l_finger_tip" reason="Never" />
+    <disable_collisions link1="${side}_gripper_base" link2="${side}_gripper_r_finger" reason="Adjacent" />
+    <disable_collisions link1="${side}_gripper_base" link2="${side}_gripper_r_finger_tip" reason="Never" />
     <disable_collisions link1="${side}_gripper_base" link2="${side}_connector_plate_base" reason="Adjacent" />
     <disable_collisions link1="${side}_gripper_base" link2="${side}_electric_gripper_base" reason="Adjacent" />
-    <disable_collisions link1="${side}_connector_plate_base" link2="${gripper_side}_gripper_l_finger" reason="Adjacent" />
-    <disable_collisions link1="${side}_connector_plate_base" link2="${gripper_side}_gripper_l_finger_tip" reason="Never" />
-    <disable_collisions link1="${side}_connector_plate_base" link2="${gripper_side}_gripper_r_finger" reason="Adjacent" />
-    <disable_collisions link1="${side}_connector_plate_base" link2="${gripper_side}_gripper_r_finger_tip" reason="Never" />
+    <disable_collisions link1="${side}_connector_plate_base" link2="${side}_gripper_l_finger" reason="Adjacent" />
+    <disable_collisions link1="${side}_connector_plate_base" link2="${side}_gripper_l_finger_tip" reason="Never" />
+    <disable_collisions link1="${side}_connector_plate_base" link2="${side}_gripper_r_finger" reason="Adjacent" />
+    <disable_collisions link1="${side}_connector_plate_base" link2="${side}_gripper_r_finger_tip" reason="Never" />
     <disable_collisions link1="${side}_electric_gripper_base" link2="${side}_connector_plate_base" reason="Adjacent" />
-    <disable_collisions link1="${side}_electric_gripper_base" link2="${gripper_side}_gripper_l_finger" reason="Adjacent" />
-    <disable_collisions link1="${side}_electric_gripper_base" link2="${gripper_side}_gripper_l_finger_tip" reason="Never" />
-    <disable_collisions link1="${side}_electric_gripper_base" link2="${gripper_side}_gripper_r_finger" reason="Adjacent" />
-    <disable_collisions link1="${side}_electric_gripper_base" link2="${gripper_side}_gripper_r_finger_tip" reason="Never" />
-    <disable_collisions link1="${side}_gripper" link2="${gripper_side}_gripper_l_finger" reason="Default" />
-    <disable_collisions link1="${side}_gripper" link2="${gripper_side}_gripper_l_finger_tip" reason="Never" />
-    <disable_collisions link1="${side}_gripper" link2="${gripper_side}_gripper_r_finger" reason="Default" />
-    <disable_collisions link1="${side}_gripper" link2="${gripper_side}_gripper_r_finger_tip" reason="Never" />
-    <disable_collisions link1="${gripper_side}_gripper_l_finger" link2="${gripper_side}_gripper_l_finger_tip" reason="Adjacent" />
-    <disable_collisions link1="${gripper_side}_gripper_l_finger" link2="${gripper_side}_gripper_r_finger" reason="Never" />
-    <disable_collisions link1="${gripper_side}_gripper_l_finger" link2="${gripper_side}_gripper_r_finger_tip" reason="Never" />
-    <disable_collisions link1="${gripper_side}_gripper_l_finger" link2="${side}_hand" reason="Never" />
-    <disable_collisions link1="${gripper_side}_gripper_l_finger" link2="${side}_hand_camera" reason="Never" />
-    <disable_collisions link1="${gripper_side}_gripper_l_finger_tip" link2="${gripper_side}_gripper_r_finger" reason="Never" />
-    <disable_collisions link1="${gripper_side}_gripper_l_finger_tip" link2="${side}_hand" reason="Never" />
-    <disable_collisions link1="${gripper_side}_gripper_l_finger_tip" link2="${side}_hand_camera" reason="Never" />
-    <disable_collisions link1="${gripper_side}_gripper_l_finger_tip" link2="${side}_wrist" reason="Never" />
-    <disable_collisions link1="${gripper_side}_gripper_r_finger" link2="${gripper_side}_gripper_r_finger_tip" reason="Adjacent" />
-    <disable_collisions link1="${gripper_side}_gripper_r_finger" link2="${side}_hand" reason="Never" />
-    <disable_collisions link1="${gripper_side}_gripper_r_finger" link2="${side}_hand_camera" reason="Never" />
-    <disable_collisions link1="${gripper_side}_gripper_r_finger" link2="${side}_wrist" reason="Never" />
-    <disable_collisions link1="${gripper_side}_gripper_r_finger_tip" link2="${side}_hand" reason="Never" />
-    <disable_collisions link1="${gripper_side}_gripper_r_finger_tip" link2="${side}_hand_camera" reason="Never" />
-    <disable_collisions link1="${gripper_side}_gripper_r_finger_tip" link2="${side}_wrist" reason="Never" />
-    <disable_collisions link1="${gripper_side}_gripper_l_finger_tip" link2="${gripper_side}_gripper_r_finger_tip" reason="Never" />
-    <disable_collisions link1="${gripper_side}_gripper_l_finger" link2="${gripper_side}_gripper_l_finger_tip" reason="Never" />
-    <disable_collisions link1="${gripper_side}_gripper_r_finger" link2="${gripper_side}_gripper_r_finger_tip" reason="Never" />
-    </xacro:if>
+    <disable_collisions link1="${side}_electric_gripper_base" link2="${side}_gripper_l_finger" reason="Adjacent" />
+    <disable_collisions link1="${side}_electric_gripper_base" link2="${side}_gripper_l_finger_tip" reason="Never" />
+    <disable_collisions link1="${side}_electric_gripper_base" link2="${side}_gripper_r_finger" reason="Adjacent" />
+    <disable_collisions link1="${side}_electric_gripper_base" link2="${side}_gripper_r_finger_tip" reason="Never" />
+    <disable_collisions link1="${side}_gripper_tip" link2="${side}_gripper_l_finger" reason="Default" />
+    <disable_collisions link1="${side}_gripper_tip" link2="${side}_gripper_l_finger_tip" reason="Never" />
+    <disable_collisions link1="${side}_gripper_tip" link2="${side}_gripper_r_finger" reason="Default" />
+    <disable_collisions link1="${side}_gripper_tip" link2="${side}_gripper_r_finger_tip" reason="Never" />
+    <disable_collisions link1="${side}_gripper_l_finger" link2="${side}_gripper_l_finger_tip" reason="Adjacent" />
+    <disable_collisions link1="${side}_gripper_l_finger" link2="${side}_gripper_r_finger" reason="Never" />
+    <disable_collisions link1="${side}_gripper_l_finger" link2="${side}_gripper_r_finger_tip" reason="Never" />
+    <disable_collisions link1="${side}_gripper_l_finger" link2="${side}_hand" reason="Never" />
+    <disable_collisions link1="${side}_gripper_l_finger" link2="${side}_hand_camera" reason="Never" />
+    <disable_collisions link1="${side}_gripper_l_finger_tip" link2="${side}_gripper_r_finger" reason="Never" />
+    <disable_collisions link1="${side}_gripper_l_finger_tip" link2="${side}_hand" reason="Never" />
+    <disable_collisions link1="${side}_gripper_l_finger_tip" link2="${side}_hand_camera" reason="Never" />
+    <disable_collisions link1="${side}_gripper_l_finger_tip" link2="${side}_wrist" reason="Never" />
+    <disable_collisions link1="${side}_gripper_r_finger" link2="${side}_gripper_r_finger_tip" reason="Adjacent" />
+    <disable_collisions link1="${side}_gripper_r_finger" link2="${side}_hand" reason="Never" />
+    <disable_collisions link1="${side}_gripper_r_finger" link2="${side}_hand_camera" reason="Never" />
+    <disable_collisions link1="${side}_gripper_r_finger" link2="${side}_wrist" reason="Never" />
+    <disable_collisions link1="${side}_gripper_r_finger_tip" link2="${side}_hand" reason="Never" />
+    <disable_collisions link1="${side}_gripper_r_finger_tip" link2="${side}_hand_camera" reason="Never" />
+    <disable_collisions link1="${side}_gripper_r_finger_tip" link2="${side}_wrist" reason="Never" />
+    <disable_collisions link1="${side}_gripper_l_finger_tip" link2="${side}_gripper_r_finger_tip" reason="Never" />
+    <disable_collisions link1="${side}_gripper_l_finger" link2="${side}_gripper_l_finger_tip" reason="Never" />
+    <disable_collisions link1="${side}_gripper_r_finger" link2="${side}_gripper_r_finger_tip" reason="Never" />
     </xacro:macro>
 </robot>

File: sawyer_moveit_config/srdf/sawyer.srdf.xacro (robot description, xacro)
@@ -2,5 +2,5 @@
 <robot name="sawyer" xmlns:xacro="http://www.ros.org/wiki/xacro">
   <!--SRDF Xacro Args-->
-  <xacro:arg name="tip_name" default="right_gripper"/>
+  <xacro:arg name="tip_name" default="right_hand"/>
   <xacro:arg name="electric_gripper" default="false"/>
   <xacro:arg name="controller_box" default="true"/>
