Commit message: Cleanup and restructure the launch with param

File: sawyer_moveit_config/srdf/rethink_clicksmart_gripper.srdf.xacro (robot description, xacro)
@@ -5,9 +5,9 @@
 -->
 <robot xmlns:xacro="http://www.ros.org/wiki/xacro" name="rethink_clicksmart_gripper">
-    <xacro:macro name="rethink_clicksmart_gripper" params="side">
-    <disable_collisions link1="${side}_l6" link2="stp_device_name_base" reason="Adjacent" />
-    <disable_collisions link1="stp_device_name_base" link2="stp_device_name_tip" reason="Adjacent" />
-    <disable_collisions link1="stp_device_name_tip" link2="${side}_hand" reason="Adjacent" />
-    <disable_collisions link1="${side}_hand" link2="stp_device_name_base" reason="Adjacent" />
+    <xacro:macro name="rethink_clicksmart_gripper" params="side stp_device_name">
+    <disable_collisions link1="${side}_l6" link2="${stp_device_name}_base" reason="Adjacent" />
+    <disable_collisions link1="${stp_device_name}_base" link2="${stp_device_name}_tip" reason="Adjacent" />
+    <disable_collisions link1="${stp_device_name}_tip" link2="${side}_hand" reason="Adjacent" />
+    <disable_collisions link1="${side}_hand" link2="${stp_device_name}_base" reason="Adjacent" />
     </xacro:macro>
 </robot>

File: sawyer_moveit_config/srdf/sawyer.srdf.xacro (robot description, xacro)
@@ -3,4 +3,5 @@
   <!--SRDF Xacro Args-->
   <xacro:arg name="tip_name" default="right_hand"/>
+  <xacro:arg name="stp_device_name" default="stp_device_name"/>
   <xacro:arg name="electric_gripper" default="false"/>
   <xacro:arg name="clicksmart_gripper" default="false"/>
@@ -21,5 +22,5 @@
   <xacro:if value="$(arg clicksmart_gripper)">
     <xacro:include filename="$(find sawyer_moveit_config)/srdf/rethink_clicksmart_gripper.srdf.xacro" />
-    <xacro:rethink_clicksmart_gripper side="right"/>
+    <xacro:rethink_clicksmart_gripper side="right" stp_device_name="$(arg stp_device_name)"/>
   </xacro:if>
 </robot>
